File: KiCad/STS BGA Beam 4.5 inch.kicad_pcb (KiCad board)
At the start: 2 copper layers, 25.4 x 114.3 mm, 20 parts

Commit message: KiCad Update
Routing:
- net (no net): track 474.7 -> 471.1 mm
Other:
- board text added: "ARTS-Lab University of South Carolina STBeam BGA V0.1 July 2025 Trotter Roberts, Ryan Yount"
- board text removed: "ARTS-Lab University of South Carolina STBeam BGA V1.0 July 2025 Trotter Roberts, Ryan Yount"
